File: eagle-t1-b/main.brd (EAGLE design)
At the start: 67 x 68.6 mm, 36 parts, among them J1 MOLEX-KK-254-2-HEADER, J10 FTSH-112-01-L-D-RA, J11 JST-PH_3-PIN-HEADER-SIDE-ENTRY, J12 JST-PH_3-PIN-HEADER-SIDE-ENTRY, J13 JST-PH_3-PIN-HEADER-SIDE-ENTRY, J14 JST-PH_4-PIN_HEADER, J15 MOLEX-KK-254-2-HEADER, J2 JST-PH_2-PIN_HEADER, J3 JST-PH_4-PIN_HEADER, J4 MOLEX-KK-254-2-HEADER-SIDE-EN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

Commit message: Finalized circuit board designs.
Parts:
- moved J4 0.63 mm to (54.0, 62.2)
- moved J5 0.63 mm to (54.0, 54.6)
- moved J11 0.38 mm to (60.6, 25.4)
- moved J12 0.38 mm to (60.6, 15.2)
- moved J13 0.38 mm to (60.6, 5.08)
Routing:
- net BBB_P9_3: track 210.3 -> 209.1 mm
- net N$4: track 23.4 -> 22.8 mm
- net N$6: track 14.3 -> 13.6 mm
- net N$5: track 16.5 -> 15.9 mm
- net N$3: track 28.5 -> 27.8 mm
